File: pcb/h_attiny10_programmer.kicad_pcb (KiCad board)
At the start: 2 copper layers, 52 parts, among them J1 PWR, J2 Conn_01x03, J3 Conn_01x03, J4 Conn_01x03, J5 Conn_01x03, J6 Conn_01x03, J7 Conn_01x03, J8 AVR-TPI-6, Q1 2N3906, SW1 SW_Push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

Commit message: pcb layout
Parts:
- added H1: M3, MountingHole:MountingHole_3.5mm, F.Cu at (104.0, 54.0)
- added H2: M3, MountingHole:MountingHole_3.5mm, F.Cu at (104.0, 126.0)
- added H3: M3, MountingHole:MountingHole_3.5mm, F.Cu at (196.0, 54.0)
- added H4: M3, MountingHole:MountingHole_3.5mm, F.Cu at (196.0, 126.0)
- added JP10: Jumper, Connector_PinHeader_2.54mm:PinHeader_1x02_P2.54mm_Vertical, F.Cu at (184.8, 103.5)
- added JP7: Jumper, Connector_PinHeader_2.54mm:PinHeader_1x02_P2.54mm_Vertical, F.Cu at (172.8, 103.5)
- added JP8: Jumper, Connector_PinHeader_2.54mm:PinHeader_1x02_P2.54mm_Vertical, F.Cu at (176.8, 103.5)
- added JP9: Jumper, Connector_PinHeader_2.54mm:PinHeader_1x02_P2.54mm_Vertical, F.Cu at (180.8, 103.5)
- C1, C4, L1, U1: moved to B.Cu
- C5, C6: footprint Capacitor_THT:C_Disc_D4.3mm_W1.9mm_P5.00mm -> Capacitor_SMD:C_0805_2012Metric_Pad1.18x1.45mm_HandSolder; moved to B.Cu
- J1: footprint Connector_PinHeader_2.54mm:PinHeader_1x02_P2.54mm_Vertical -> TerminalBlock:TerminalBlock_bornier-2_P5.08mm
- U4: footprint Package_TO_SOT_SMD:SOT-23-6 -> Package_DIP:DIP-6_W7.62mm
- moved R15 181.1 mm to (180.0, 113.7)
- moved R12 180.9 mm to (177.6, 113.7), turned to 180 degrees
- moved R13 175.2 mm to (177.5, 109.8), turned to 180 degrees
- moved R11 171.2 mm to (187.2, 96.9), turned to 180 degrees
- moved R14 169.6 mm to (180.1, 109.8)
- moved R10 166.6 mm to (177.0, 93.2)
- moved R3 165.3 mm to (184.2, 70.5), turned to 180 degrees
- moved D1 164.8 mm to (174.0, 80.5)
- moved R5 164.6 mm to (184.2, 59.5), turned to 180 degrees
- moved R9 155.9 mm to (187.2, 89.4), turned to 180 degrees
- moved R1 152.9 mm to (184.2, 62.9), turned to 180 degrees
- moved R2 147.3 mm to (174.0, 77.0)
- moved R8 146.4 mm to (163.5, 70.9), turned to 270 degrees
- moved D6 144.7 mm to (180.8, 118.8)
- moved D7 137.2 mm to (187.4, 118.8)
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Connections:
- net /CLK renamed CLK
- net /DATA renamed DATA
- net /PROG_12V renamed PROG_12V
- net /RESET renamed RESET
- J4 pad 1: /PB0 -> PB0
- J4 pad 2: /PB0 -> PB0
- J4 pad 3: /PB0 -> PB0
- J5 pad 1: /PB1 -> PB1
- J5 pad 2: /PB1 -> PB1
- J5 pad 3: /PB1 -> PB1
- J6 pad 1: /PB2 -> PB2
- J6 pad 2: /PB2 -> PB2
- J6 pad 3: /PB2 -> PB2
- J7 pad 1: /PB3 -> PB3
- J7 pad 2: /PB3 -> PB3
- J7 pad 3: /PB3 -> PB3
- JP4 pad 3: /PB0 -> PB0
- JP5 pad 3: /PB1 -> PB1
- JP6 pad 3: /PB3 -> PB3
- R12 pad 1: /PB0 -> Net-(JP7-Pad2)
- R13 pad 1: /PB1 -> Net-(JP8-Pad2)
- R14 pad 1: /PB2 -> Net-(JP9-Pad2)
- R15 pad 1: /PB3 -> Net-(JP10-Pad2)
- SW1 pad 1: /PB0 -> PB0
- SW2 pad 1: /PB1 -> PB1
- SW3 pad 1: /PB2 -> PB2
- SW4 pad 1: /PB3 -> PB3
- U4 pad 4: /PB2 -> PB2
Routing:
- net +5V: track 0.00 -> 234.2 mm
- net Vin: track 0.00 -> 129.3 mm
- net PB2: track 0.00 -> 103.3 mm
- net PB0: track 0.00 -> 103.0 mm
- net PB3: track 0.00 -> 102.0 mm
- net PB1: track 0.00 -> 92.6 mm
- net dcdc_12V: track 0.00 -> 55.1 mm
- net PROG_12V: track 0.00 -> 33.9 mm
- net CLK: track 0.00 -> 28.5 mm
- net Net-(JP4-Pad2): track 0.00 -> 26.0 mm
- net GND: track 0.00 -> 22.8 mm
- net Net-(D1-Pad2): track 0.00 -> 21.1 mm
- net RESET: track 0.00 -> 16.7 mm
- net DATA: track 0.00 -> 16.4 mm
- net Net-(C3-Pad1): track 0.00 -> 15.6 mm
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- added copper zone on B.Cu, net GND
Other:
- board outline added: 100 x 80 mm

Commit message: clean up layout
Parts:
- moved Q1 3.07 mm to (176.5, 86.0)
- moved R10 3.07 mm to (174.1, 94.2)
- moved R11 3.07 mm to (184.3, 97.9)
- moved R9 3.07 mm to (184.3, 90.4)
Routing:
- net GND: track 22.8 -> 10.5 mm
- net Vin: track 129.3 -> 119.5 mm
- net Net-(D1-Pad2): track 21.1 -> 29.9 mm
- net +5V: track 234.2 -> 227.6 mm
- net PROG_12V: track 33.9 -> 30.6 mm
- net Net-(R10-Pad1): track 11.3 -> 8.59 mm
